Commit message: add lidar e camera no xacro

File: ugv_embrapa_ws/install/osr_gazebo/share/osr_gazebo/urdf/gazebo.urdf.xacro (robot description, xacro)
@@ -137,3 +137,54 @@
         </sensor>
     </gazebo>
+      <!--Lidar-->
+    <gazebo reference="lidar_link">
+      <sensor name="laser" type="ray">
+        <pose> 0 0 0 0 0 0 </pose>
+        <visualize>true</visualize>
+        <update_rate>10</update_rate>
+        <ray>
+          <scan>
+            <horizontal>
+              <samples>360</samples>
+              <min_angle>-3.14</min_angle>
+              <max_angle>3.14</max_angle>
+            </horizontal>
+          </scan>
+          <range>
+            <min>0.3</min>
+            <max>12</max>
+          </range>
+        </ray>
+        <plugin name="laser_controller" filename="libgazebo_ros_ray_sensor.so">
+          <ros>
+            <argument>~/out:=scan</argument>
+          </ros>
+          <output_type>sensor_msgs/LaserScan</output_type>
+          <frame_name>lidar_link</frame_name>
+        </plugin>
+      </sensor>
+    </gazebo>
+    <!-- Camera-->
+    <gazebo reference="camera_link">
+          <sensor name="camera" type="camera">
+              <pose> 0 0 0 0 0 0 </pose>
+              <visualize>true</visualize>
+              <update_rate>10</update_rate>
+              <camera>
+                  <horizontal_fov>1.089</horizontal_fov>
+                  <image>
+                      <format>R8G8B8</format>
+                      <width>640</width>
+                      <height>480</height>
+                  </image>
+                  <clip>
+                      <near>0.05</near>
+                      <far>8.0</far>
+                  </clip>
+              </camera>
+              <plugin name="camera_controller" filename="libgazebo_ros_camera.so">
+                  <frame_name>camera_link</frame_name>
+              </plugin>
+          </sensor>
+      </gazebo>
 </robot>

File: ugv_embrapa_ws/install/osr_gazebo/share/osr_gazebo/urdf/osr.urdf.xacro (robot description, xacro)
@@ -426,4 +426,24 @@
         </joint>
     <link name="imu_link"></link>
+    <!-- Lidar -->
+    <link name="lidar_link">
+        <visual>
+        <origin xyz="0 0 0" rpy="0 0 0"/>
+        <geometry>
+            <cylinder length="0.03" radius="0.03"/>
+        </geometry>
+        </visual>
+        <collision>
+        <origin xyz="0 0 0" rpy="0 0 0"/>
+        <geometry>
+            <cylinder length="0.03" radius="0.03"/>
+        </geometry>
+        </collision>
+    </link>
+    <joint name="lidar_joint" type="fixed">
+        <origin xyz="0.1 0 0.080" rpy="0 0 0"/>
+        <parent link="base_link"/>
+        <child link="lidar_link"/>
+    </joint>
     <xacro:insert_velocity_transmission name="rear_wheel_joint_right"/>
     <xacro:insert_velocity_transmission name="rear_wheel_joint_left"/>
